Commit message: updated readme

File: racecar_gazebo/racecar_description/urdf/_d435.urdf.xacro (robot description, xacro)
@@ -48,6 +48,6 @@
         <geometry>
           <!-- <box size="${d435_cam_width} ${d435_cam_height} ${d435_cam_depth}"/> -->
-          <mesh filename="package://realsense2_description/meshes/d435.dae" />
-          <!--<mesh filename="package://realsense2_description/meshes/d435/d435.dae" />-->
+          <mesh filename="package://racecar_description/meshes/d435.dae" />
+          <!--<mesh filename="package://racecar_description/meshes/d435/d435.dae" />-->
         </geometry>
         <material name="${name}_aluminum"/>

Commit message: added kinect to robot, still   zed oooooooutput

File: racecar_gazebo/racecar_description/urdf/_d435.urdf.xacro (robot description, xacro)
@@ -47,5 +47,5 @@
       <origin xyz="${d435_cam_mount_from_center_offset} ${-d435_cam_depth_py} 0" rpy="${M_PI/2} 0 ${M_PI/2}"/>
         <geometry>
-          <!-- <box size="${d435_cam_width} ${d435_cam_height} ${d435_cam_depth}"/> -->
+    <!--       <box size="${d435_cam_width} ${d435_cam_height} ${d435_cam_depth}"/> -->
           <mesh filename="package://racecar_description/meshes/d435.dae" />
           <!--<mesh filename="package://racecar_description/meshes/d435/d435.dae" />-->

File: racecar_gazebo/racecar_description/urdf/racecar.xacro (robot description, xacro)
@@ -146,4 +146,5 @@
   <xacro:wheel_transmission name="right_front_wheel" />
   <!-- Add Hokuyo laser scanner -->
+<!--
   <link name="laser">
     <inertial>
@@ -170,7 +171,82 @@
     <axis xyz="0 0 1" />
   </joint>
-  <!-- zed camera -->
+-->
+<!-- Camera
+<xacro:include filename="$(find kinect_description)/urdf/kinect.urdf.xacro" />
+-->
+<link name="camera_link">
+  <inertial>
+      <mass value="1e-5" />
+      <origin xyz="0 0 0" rpy="0 0 0"/>
+      <inertia ixx="1e-6" ixy="0" ixz="0" iyy="1e-6" iyz="0" izz="1e-6" />
+    </inertial>
+  <collision name="collision">
+    <geometry>
+      <box size="0.073000 0.276000 0.072000" />
+    </geometry>
+  </collision>
+  <visual name="visual">
+    <geometry>
+      <mesh filename="package://racecar_description/meshes/kinect.dae"/>
+    </geometry>
+  </visual>
+  <sensor name="camera" type="depth">
+    <update_rate>20</update_rate>
+    <camera>
+      <horizontal_fov>1.047198</horizontal_fov>
+      <image>
+        <width>640</width>
+        <height>480</height>
+        <format>R8G8B8</format>
+      </image>
+      <clip>
+        <near>0.05</near>
+        <far>7</far>
+          </clip>
+        </camera>
+        <plugin name="camera_plugin" filename="libgazebo_ros_openni_kinect.so">
+          <baseline>0.2</baseline>
+          <alwaysOn>true</alwaysOn>
+          <!-- Keep this zero, update_rate in the parent <sensor> tag
+            will control the frame rate.-->
+          <updateRate>0.0</updateRate>
+          <cameraName>camera_ir</cameraName>
+          <imageTopicName>/camera/color/image_raw</imageTopicName>
+          <cameraInfoTopicName>/camera/color/camera_info</cameraInfoTopicName>
+          <depthImageTopicName>/camera/depth/image_raw</depthImageTopicName>
+          <depthImageCameraInfoTopicName>/camera/depth/camera_info</depthImageCameraInfoTopicName>
+          <pointCloudTopicName>/camera/depth/points</pointCloudTopicName>
+          <frameName>chassis</frameName>
+          <pointCloudCutoff>0.5</pointCloudCutoff>
+          <pointCloudCutoffMax>7.0</pointCloudCutoffMax>
+          <distortionK1>0</distortionK1>
+          <distortionK2>0</distortionK2>
+          <distortionK3>0</distortionK3>
+          <distortionT1>0</distortionT1>
+          <distortionT2>0</distortionT2>
+          <CxPrime>0</CxPrime>
+          <Cx>0</Cx>
+          <Cy>0</Cy>
+          <focalLength>0</focalLength>
+          <hackBaseline>0</hackBaseline>
+        </plugin>
+      </sensor>
+    </link>
+    <joint name="depth_camera_joint" type="fixed">
+      <origin xyz="0.390 0 0.04" rpy="0 0 0"/>
+      <parent link="chassis"/>
+      <child link="camera_link"/>
+      <axis xyz="0 0 1" />
+       <limit lower="0.0" upper="0.0" effort="0.0" velocity="0.0" />
+    </joint>
+    <!--
+<xacro:kinect name="camera" parent="chassis">
+  <origin xyz="-0.02 0 -0.04" rpy="0 -1.60 0" />
+  <inertia ixx="0.1" ixy="0" ixz="0" iyy="0.1" iyz="0" izz="0.1" />
+</xacro:kinect>
+-->
+<!--   zed camera
   <link name="zed_camera_link">
-    <inertial>
+  <inertial>
       <mass value="1e-5" />
       <origin xyz="0 0 0" rpy="0 0 0"/>
@@ -196,9 +272,9 @@
     <child link="zed_camera_link"/>
     <axis xyz="0 0 1" />
-    <!-- <limit lower="0.0" upper="0.0" effort="0.0" velocity="0.0" /> -->
-  </joint>
-  <!-- zed camera lenses -->
-  <!-- It seems these have to have a non-zero mass to have a camera attached? -->
-  <link name="camera_link"><!-- this needs to match the name in zed_wrapper/zed_tf.launch -->
+     <limit lower="0.0" upper="0.0" effort="0.0" velocity="0.0" />
+  </joint>
+ zed camera lenses
+ It seems these have to have a non-zero mass to have a camera attached?
+  <link name="camera_link"><this needs to match the name in zed_wrapper/zed_tf.launch
     <inertial>
       <mass value="1e-5" />
@@ -226,11 +302,7 @@
     <axis xyz="0 0 1" />
   </joint>
+-->
   <!-- Add the remaining xacros -->
   <xacro:include filename="$(find racecar_description)/urdf/racecar.gazebo" />
   <xacro:include filename="$(find racecar_description)/urdf/materials.xacro" />
-  <xacro:include filename="$(find racecar_description)/urdf/_d435.urdf.xacro">
-    <sensor_d435 parent="${prefix}base_link">
-      <origin xyz="0.0 0.2 0" rpy="0 0 0"/>
-    </sensor_d435>
-  </xacro:include>
 </robot>
