Commit message: added realsense not working

File: racecar_gazebo/racecar_description/urdf/racecar.xacro (robot description, xacro)
@@ -229,3 +229,8 @@
   <xacro:include filename="$(find racecar_description)/urdf/racecar.gazebo" />
   <xacro:include filename="$(find racecar_description)/urdf/materials.xacro" />
+  <xacro:include filename="$(find racecar_description)/urdf/_d435.urdf.xacro">
+    <sensor_d435 parent="${prefix}base_link">
+      <origin xyz="0.0 0.2 0" rpy="0 0 0"/>
+    </sensor_d435>
+  </xacro:include>
 </robot>

Commit message: Working depth pointcloud

File: racecar_gazebo/racecar_description/urdf/racecar.xacro (robot description, xacro)
@@ -146,5 +146,4 @@
   <xacro:wheel_transmission name="right_front_wheel" />
   <!-- Add Hokuyo laser scanner -->
-<!--
   <link name="laser">
     <inertial>
@@ -171,80 +170,5 @@
     <axis xyz="0 0 1" />
   </joint>
--->
-<!-- Camera
-<xacro:include filename="$(find kinect_description)/urdf/kinect.urdf.xacro" />
--->
-<link name="camera_link">
-  <inertial>
-      <mass value="1e-5" />
-      <origin xyz="0 0 0" rpy="0 0 0"/>
-      <inertia ixx="1e-6" ixy="0" ixz="0" iyy="1e-6" iyz="0" izz="1e-6" />
-    </inertial>
-  <collision name="collision">
-    <geometry>
-      <box size="0.073000 0.276000 0.072000" />
-    </geometry>
-  </collision>
-  <visual name="visual">
-    <geometry>
-      <mesh filename="package://racecar_description/meshes/kinect.dae"/>
-    </geometry>
-  </visual>
-  <sensor name="camera" type="depth">
-    <update_rate>20</update_rate>
-    <camera>
-      <horizontal_fov>1.047198</horizontal_fov>
-      <image>
-        <width>640</width>
-        <height>480</height>
-        <format>R8G8B8</format>
-      </image>
-      <clip>
-        <near>0.05</near>
-        <far>7</far>
-          </clip>
-        </camera>
-        <plugin name="camera_plugin" filename="libgazebo_ros_openni_kinect.so">
-          <baseline>0.2</baseline>
-          <alwaysOn>true</alwaysOn>
-          <!-- Keep this zero, update_rate in the parent <sensor> tag
-            will control the frame rate.-->
-          <updateRate>0.0</updateRate>
-          <cameraName>camera_ir</cameraName>
-          <imageTopicName>/camera/color/image_raw</imageTopicName>
-          <cameraInfoTopicName>/camera/color/camera_info</cameraInfoTopicName>
-          <depthImageTopicName>/camera/depth/image_raw</depthImageTopicName>
-          <depthImageCameraInfoTopicName>/camera/depth/camera_info</depthImageCameraInfoTopicName>
-          <pointCloudTopicName>/camera/depth/points</pointCloudTopicName>
-          <frameName>chassis</frameName>
-          <pointCloudCutoff>0.5</pointCloudCutoff>
-          <pointCloudCutoffMax>7.0</pointCloudCutoffMax>
-          <distortionK1>0</distortionK1>
-          <distortionK2>0</distortionK2>
-          <distortionK3>0</distortionK3>
-          <distortionT1>0</distortionT1>
-          <distortionT2>0</distortionT2>
-          <CxPrime>0</CxPrime>
-          <Cx>0</Cx>
-          <Cy>0</Cy>
-          <focalLength>0</focalLength>
-          <hackBaseline>0</hackBaseline>
-        </plugin>
-      </sensor>
-    </link>
-    <joint name="depth_camera_joint" type="fixed">
-      <origin xyz="0.390 0 0.04" rpy="0 0 0"/>
-      <parent link="chassis"/>
-      <child link="camera_link"/>
-      <axis xyz="0 0 1" />
-       <limit lower="0.0" upper="0.0" effort="0.0" velocity="0.0" />
-    </joint>
-    <!--
-<xacro:kinect name="camera" parent="chassis">
-  <origin xyz="-0.02 0 -0.04" rpy="0 -1.60 0" />
-  <inertia ixx="0.1" ixy="0" ixz="0" iyy="0.1" iyz="0" izz="0.1" />
-</xacro:kinect>
--->
-<!--   zed camera
+   zed camera
   <link name="zed_camera_link">
   <inertial>
@@ -274,7 +198,7 @@
      <limit lower="0.0" upper="0.0" effort="0.0" velocity="0.0" />
   </joint>
- zed camera lenses
- It seems these have to have a non-zero mass to have a camera attached?
-  <link name="camera_link"><this needs to match the name in zed_wrapper/zed_tf.launch
+ <!--zed camera lenses
+ It seems these have to have a non-zero mass to have a camera attached?-->
+  <link name="camera_link"> <!--this needs to match the name in zed_wrapper/zed_tf.launch-->
     <inertial>
       <mass value="1e-5" />
@@ -302,5 +226,4 @@
     <axis xyz="0 0 1" />
   </joint>
--->
   <!-- Add the remaining xacros -->
   <xacro:include filename="$(find racecar_description)/urdf/racecar.gazebo" />

Commit message: added IMU

File: racecar_gazebo/racecar_description/urdf/racecar.xacro (robot description, xacro)
@@ -226,4 +226,30 @@
     <axis xyz="0 0 1" />
   </joint>
+  <!-- Add imu -->
+  <link name="imu_link">
+    <inertial>
+      <mass value="0.05" />
+      <inertia ixx="4e-6" ixy="0" ixz="0" iyy="4e-6" iyz="0" izz="4e-6" />
+    </inertial>
+    <collision>
+      <origin xyz="0 0 0" rpy="0 0 0"/>
+      <geometry>
+        <box size="0.03 0.03 0.03"/>
+      </geometry>
+    </collision>
+    <visual>
+      <origin xyz="0 0 0" rpy="0 0 0"/>
+      <geometry>
+        <box size="0.03 0.03 0.03"/>
+      </geometry>
+      <material name="orange" />
+    </visual>
+  </link>
+  <joint name="imu_joint" type="fixed">
+    <origin xyz="0.265 0.0 0.0" rpy="0 0 0"/>
+    <parent link="chassis" />
+    <child link="imu_link" />
+    <axis xyz="0 0 1" />
+  </joint>
   <!-- Add the remaining xacros -->
   <xacro:include filename="$(find racecar_description)/urdf/racecar.gazebo" />
